File: khellen/khellen.kicad_sch (KiCad schematic)
At the start: 80 parts, among them J1 1318612-1, J2 AudioJack3_SwitchTR, M1 Module-mega-mcu144-0.7, M2 Module-output-0.3, M3 Module-wbo-0.5, M4 Module-power_12and5V-0.3, M5 Module-knock-0.2, M6 Module-lin-0.1, M7 Module-stlink-0.1, M8 Module-ign8-0.2, P1 Pad, P10 Pad, P11 Pad, P12 Pad, P13 Pad, P14 Pad, P15 Pad, P16 Pad, P17 Pad, P18 Pad, P19 Pad, P2 Pad, P20 Pad, P21 Pad, P22 Pad, P23 Pad, P24 Pad, P25 Pad, P26 Pad, P27 Pad, P28 Pad, P29 Pad, P3 Pad, P30 Pad, P31 Pad, P32 Pad, P33 Pad, P34 Pad, P35 Pad, P36 Pad, P37 Pad, P38 Pad, P40 Pad, P41 Pad, P42 Pad, P43 Pad, P44 Pad, P45 Pad, P46 Pad, P47 Pad, P48 Pad, P49 Pad, P50 Pad, P51 Pad, P52 Pad, P53 Pad, P54 Pad, P55 Pad, P6 Pad, P7 Pad, P8 Pad, P89 Pad, P9 Pad, P90 Pad, P91 Pad, P92 Pad, U1 TLE9201SG, U2 DG470, U3 MCP6002-xSN

Commit message: Updated PCB, updated schematic
Parts:
- removed BT1: DNP, symbol Device:Battery_Cell
- removed C1: 100n, symbol Device:C
- removed C2: 10u, symbol Device:C
- removed J2: AudioJack3_SwitchTR, symbol Connector_Audio:AudioJack3_SwitchTR
- removed P1, P10, P11, P12, P13, P14, P15, P16, P17, P18, P19, P2, P20, P21, P22, P23, P24, P25, P26, P27, P28, P29, P3, P30, P31, P32, P33, P34, P35, P36, P37, P38, P40, P41, P42, P43, P44, P45, P46, P47, P48, P49, P50, P51, P52, P53, P54, P55, P6, P7, P8, P89, P90, P91, P92: Pad, hellen-one-common:PAD-TH, symbol hellen-one-common:Pad
- removed R2, R3, R4: Jumper-Pad-Pad, hellen-one-common:PAD-0805-PAD, symbol hellen-one-common:Jumper-Pad-Pad
- removed U3: MCP6002-xSN, symbol Amplifier_Operational:MCP6002-xSN
- added C12: 10n, Capacitor_SMD:C_0402_1005Metric, symbol Device:C
- added C13: 10u, Capacitor_SMD:C_0402_1005Metric, symbol Device:C
- added C14, C3: 100n, Capacitor_SMD:C_0402_1005Metric, symbol Device:C
- added D10, D11, D12, D2, D3, D4, D5, D6, D7, D8, D9: SS34, Diode_SMD:D_SMA, symbol Diode:SS34
- added D13, D16, D18, D20, D25, D26, D27, D28, D33, D34, D36, D41, D42, D43, D44, D49, D50, D51, D52: LED_0603, LED_SMD:LED_0603_1608Metric, symbol misc:LED_0603
- added D14, D15, D17, D19, D21, D22, D23, D24, D29, D30, D32, D37, D38, D39, D40, D45, D46, D47, D48: 1N4148WS, Diode_SMD:D_SOD-323, symbol Diode:1N4148WS
- added J3: USB_B, Connector_USB:USB_B_TE_5787834_Vertical, symbol misc:USB_B
- added J4: Conn_01x06, Connector_PinHeader_2.54mm:PinHeader_1x06_P2.54mm_Vertical, symbol Connector_Generic:Conn_01x06
- added J5: Conn_01x06_Pin, Connector_PinHeader_2.54mm:PinHeader_1x06_P2.54mm_Vertical, symbol Connector:Conn_01x06_Pin
- added J6: Conn_01x05_Pin, Connector_PinHeader_2.54mm:PinHeader_1x05_P2.54mm_Vertical, symbol Connector:Conn_01x05_Pin
- added P1, P10, P11, P12, P13, P15, P16, P18, P19, P2, P20, P21, P22, P23, P24, P25, P28, P29, P3, P30, P31, P32, P33, P34, P35, P37, P38, P4, P40, P44, P45, P5, P6, P7, P8, P9: Pad, kicad6-libraries:PAD-TH, symbol misc:Pad
- added Q1, Q2, Q3, Q4, Q5, Q6: VND14NV04TR-E, Package_TO_SOT_SMD:TO-252-2, symbol semiconductors:VND14NV04TR-E
- added R1, R24, R25, R26, R27, R28, R29, R31: 10k, Resistor_SMD:R_0603_1608Metric, symbol Device:R
- added R2, R35, R37, R39, R40, R41: DNP, Resistor_SMD:R_0603_1608Metric, symbol Device:R_Small
- added R3, R36, R38, R42, R43, R44: 680k, Resistor_SMD:R_0603_1608Metric, symbol Device:R_Small
- added R30, R5: 120, Resistor_SMD:R_0603_1608Metric, symbol Device:R
- added R32: 4.7k, Resistor_SMD:R_0603_1608Metric, symbol Device:R
- added R33, R6, R7: 1k, Resistor_SMD:R_0603_1608Metric, symbol Device:R
- added R34: 10k, Resistor_SMD:R_0603_1608Metric, symbol Device:R_Small
- added R45, R46, R47, R48, R49, R50, R51, R52, R53, R54, R55, R56, R57, R58, R59, R60, R61, R62, R63, R64, R65, R66, R67, R68, R69, R70, R71, R72, R73, R74, R75, R76, R77, R78, R79, R80, R81, R82, R83, R84, R85, R86, R87: 0, Resistor_SMD:R_0603_1608Metric, symbol Device:R
- added RN1, RN2: R_Pack04, Resistor_SMD:R_Array_Convex_4x0612, symbol Device:R_Pack04
- added RN3: 10k, Resistor_SMD:R_Array_Convex_4x0612, symbol Device:R_Pack04
- added RN4, RN5, RN6, RN7: 20k, Resistor_SMD:R_Array_Convex_4x0612, symbol Device:R_Pack04
- added U5: BTS6143D, Package_TO_SOT_SMD:TO-252-4, symbol Power_Management:BTS6143D
- added U6: BTS4175SGA, Package_SO:SOIC-8_3.9x4.9mm_P1.27mm, symbol EasyEDA:BTS4175SGA
- BT2: footprint (none) -> Battery:BatteryHolder_Renata_SMTU2032-LF_1x2032
- F1, F2: footprint hellen-one-common:PAD-1206-PAD -> Fuse:Fuse_0805_2012Metric
- F3: footprint hellen-one-common:PAD-1206-PAD -> Fuse:Fuse_0805_2012Metric; LCSC C182446 -> (none); MyComment (none) -> DNP
- J1: footprint kicad6-libraries:TE_1318612-1 -> khellen:TE_1318612-1
- M1: footprint hellen-one-mega-mcu144-0.7:mega-mcu144 -> khellen:mega-mcu144
- M2: footprint hellen-one-output-0.3:output -> khellen:output
- M3: footprint hellen-one-wbo-0.5:wbo -> khellen:wbo
- M4: footprint hellen-one-power_12and5V-0.3:power_12and5V -> khellen:power_12and5V
- M5: footprint hellen-one-knock-0.2:knock -> khellen:knock
- M6: footprint hellen-one-lin-0.1:lin -> khellen:lin
- M7: footprint hellen-one-stlink-0.1:stlink -> khellen:stlink
- M8: footprint hellen-one-ign8-0.2:ign8 -> khellen:ign8
- renumbered P9 to P14
Connections:
- net 12V_RAW is gone; now on net +12V_RAW: F1.2, F2.2, M4.V3 (V12_RAW)
- net OUT_IMRC is gone; now on net GNDA: J1.A11
- net +12V: now also M6.N1 (12V), M6.V1 (12V)
- net +5V: now also M2.W14 (V5), M7.N1 (V5); no longer M5.E1 (V5A)
- net +5VP: now also J1.C22, R53.2, R54.2
- net 4WIRE_DENSO_SIGNAL+: now also R46.2; no longer J1.A6
- net AIN1: now also R2.2, R3.1, R75.2
- net AIN2: now also R35.2, R36.1, R74.2
- net AIN3: now also R37.2, R38.1, R73.2
- net CAN_H: now also J1.C15, M1.W12 (CANH), M3.W4 (CANH), U2.1, J5.1 (Pin_1); no longer J1.E11
- net CAN_L: now also J1.C14, M1.W13 (CANL), M3.W3 (CANL), J5.2 (Pin_2), R5.2; no longer J1.E24
- net DC_PWM: now also U1.12 (PWM)
- net DIN1: now also R39.2, R42.1, R78.2
- net DIN2: now also R40.2, R43.1, R77.2
- net DIN3: now also R41.2, R44.1, R76.2
- net GND: now also J1.C20, J1.E3, M2.G (GND), M2.S3 (GND), M3.E6 (LSU_H-), M3.G (GND), M6.E1 (GND), M6.S1 (GND), M7.G (GND), M8.G (GND), U1.10 (SCK), U1.13 (GND), U1.6 (GND), U1.8 (SI), U1.9 (CSN), U2.3 (GND), U2.5 (~{EN}), U2.7 (V-), C12.2, C13.2, C14.2, C3.1, D12.2 (A), J3.4 (GND), J3.5 (Shield), J4.3 (Pin_3), J6.4 (Pin_4), J6.5 (Pin_5), Q1.3 (S), Q2.3 (S), Q3.3 (S), Q4.3 (S), Q5.3 (S), Q6.3 (S), R1.2, R24.2, R25.2, R26.2, R27.2, R28.2, R29.2, R30.1, R32.1, R33.2, RN1.1 (R1.1), RN1.2 (R2.1), RN1.3 (R3.1), RN1.4 (R4.1), RN2.1 (R1.1), RN2.2 (R2.1), RN2.3 (R3.1), RN2.4 (R4.1), RN6.8 (R1.2); no longer J1.A23, J1.A24, J1.A8, J1.A9, J1.E4
- net IN_BRAKE: now also R83.2; no longer J1.E22
- net IN_CLT: now also R66.2; no longer J1.B8
- net IN_IAT: now also R68.2; no longer J1.B17
- net IN_INTAKE_POSITION: now also R48.2
- net IN_KNOCK: now also R87.2; no longer J1.A1
- net IN_MAP: now also R52.2; no longer J1.A30
- net IN_TPS: now also J1.A15; no longer J1.A29
- net IN_VSS: now also R51.2; no longer J1.A18
- net IN_VTEC_PRESSURE_SW: now also R67.2
- net MCU_AUX_LS2: now also M8.V5 (IGN4), RN1.8 (R1.2)
- net MCU_AUX_LS3: now also M8.V6 (IGN3), RN1.7 (R2.2)
- net MCU_LS_EVAP: now also M8.V2 (IGN7), RN2.7 (R2.2)
- net MCU_VTC_LS: now also M8.V1 (IGN8), RN2.8 (R1.2)
- net MCU_WBO_HEATER_LOW_SIDE: now also M8.V3 (IGN6), RN2.6 (R3.2)
- net OUT_CHECK_ENGINE: now also M2.S14 (OUT_LOW9), D37.2 (A), D41.2 (K), R86.2; no longer J1.E31
- net OUT_IGN1: now also R62.2; no longer J1.A16
- net OUT_IGN2: now also R61.2; no longer J1.A15
- net OUT_IGN3: now also R60.2; no longer J1.A14
- net OUT_IGN4: now also R59.2; no longer J1.A13
- net OUT_INJ1: now also D19.2 (A), D20.2 (K)
- net OUT_INJ2: now also D17.2 (A), D18.2 (K)
- net OUT_INJ3: now also D15.2 (A), D16.2 (K)
- net OUT_INJ4: now also D13.2 (K), D14.2 (A)
- net P24: now also P24.1 (Pin_1)
- net P25: now also P25.1 (Pin_1)
- net P28: now also P28.1 (Pin_1)
- net P29: now also P29.1 (Pin_1)
- net P30: now also P30.1 (Pin_1)
- net P31: now also P31.1 (Pin_1)
- net P32: now also P32.1 (Pin_1)
- net P33: now also P33.1 (Pin_1)
- net P34: now also P34.1 (Pin_1)
- net P35: now also P35.1 (Pin_1)
- net P37: now also P37.1 (Pin_1)
- net P40: now also P40.1 (Pin_1)
- net P45: now also P45.1 (Pin_1)
- net V33_REF: now also M3.W9 (VDDA)
- net at J1.E26: now also R85.1
- net at J1.C8: now also R73.1
- net at J1.E23: now also P12.1 (Pin_1)
- net +12V_RAW: now reaches J1.C2
- net +12V_RAW: now also M2.S11 (V12_RAW), U1.4 (VS), U2.4 (V+), C13.1, C14.1, C3.2, D10.1 (K), D11.1 (K), D2.1 (K), D3.1 (K), D4.1 (K), D5.1 (K), D6.1 (K), D7.1 (K), D8.1 (K), D9.1 (K), R63.2, U5.3 (Vbb), U6.5 (VS), U6.6 (VS), U6.7 (VS), U6.8 (VS)
- net at J1.A12: now also R49.1
- net at J1.E12: now also P8.1 (Pin_1)
- net +3V3: now reaches M7.N2 (V33)
- net +3V3: now also M1.N22 (V33), M1.N32 (V33), U1.2 (VSO), R31.2, R34.2
- net at M7.N3 (SWO): now also M1.N6 (SWO)
- net at M7.N4 (SWDIO): now also M1.N7 (SWDIO)
- net at M7.N5 (SWCLK): now also M1.N8 (SWCLK)
- net at M7.N6 (nReset): now also M1.N9 (nReset)
- net at J1.E2: now also P5.1 (Pin_1)
- net at J1.E18: now also R82.1
- net at J1.A28: now also R60.1
- net at J1.C4: now also M3.E4 (LSU_Rtrim)
- net at J1.C10: now also R75.1
- net OUT_AUX_LS3: now reaches J1.C11
- net OUT_AUX_LS3: now also D6.2 (A), Q1.2 (D)
- net OUT_AUX_LS2: now reaches J1.C12
- net OUT_AUX_LS2: now also D7.2 (A), Q2.2 (D)
- net OUT_AUX_LS1: now reaches J1.C13
- net OUT_AUX_LS1: now also D9.2 (A), Q4.2 (D)
- net OUT_DCn: now reaches J1.C16
- net OUT_DCn: now also U1.5 (OUT1)
- net OUT_DCp: now reaches J1.C17
- net OUT_DCp: now also U1.7 (OUT2)
- net at J1.C18: now also R76.1
- net at J1.C19: now also R77.1
- net at J1.C21: now also R78.1
- net at J1.C3: now also M3.E1 (LSU_Un)
- net at J1.C5: now also M3.E3 (LSU_Ip)
- net at J1.C6: now also M3.E2 (LSU_Vm)
- net at J1.C7: now also M3.E5 (LSU_H+)
- net at J1.C9: now also R74.1
- net at J1.E1: now also R79.1
- net at J1.E14: now also P9.1 (Pin_1)
- net at J1.E15: now also P10.1 (Pin_1)
- net at J1.E16: now also P11.1 (Pin_1)
- net at J1.E27: now also P38.1 (Pin_1)
- net at J1.E29: now also P44.1 (Pin_1)
- net at J1.E6: now also P7.1 (Pin_1)
- net at J1.E8: now also R81.1
- net GNDA: now reaches J1.A10
- net GNDA: now also M1.E39 (GNDA), M1.W1 (GNDA), R3.2, R36.2, R38.2, R42.2, R43.2, R44.2, R55.2, R56.2
- net MCU_AUX_01: now reaches M1.E35 (IO6)
- net MCU_AUX_01: now also M8.V8 (IGN1), RN1.5 (R4.2)
- net DC_DIR: now reaches M1.E36 (IO7)
- net DC_DIR: now also U1.1 (DIR)
- net +5VA: now reaches M1.E38 (V5A_SWITCHABLE)
- net +5VA: now also M1.W2 (V5A_SWITCHABLE), M3.W1 (V5_IN), M5.E1 (V5A), M6.V3 (5V), M8.V9 (VCC), R2.1, R35.1, R37.1, R39.1, R40.1, R41.1
- net at M1.N10 (SPI3_CS): now also U2.6, R1.1
- net IO1: now reaches M1.N16 (IO1)
- net at M1.N17 (UART2_TX): now also R7.1
- net at M1.N18 (UART2_RX): now also R6.1
- net IO2: now reaches M1.N19 (IO2)
- net at M1.N2 (USBM): now also J3.2 (D-), J6.2 (Pin_2)
- net IO4: now reaches M1.N20 (IO4)
- net IO3: now reaches M1.N21 (IO3)
- net DC_DIS: now reaches M1.N23 (IO5)
- net DC_DIS: now also U1.11 (DIS), R34.1
- net MCU_AUX_02: now reaches M1.N24 (UART8_RX)
- net MCU_AUX_02: now also M8.V7 (IGN2), RN1.6 (R3.2)
- net +3.3VA: now reaches M1.N28 (V33_SWITCHABLE)
- net +3.3VA: now also M8.V10 (V33)
- net at M1.N3 (USBP): now also J3.3 (D+), J6.3 (Pin_3)
- net at M1.N4 (VBUS): now also J3.1 (VBUS), J6.1 (Pin_1)
- net DENSO/OUT: now reaches M1.S15 (IN_O2S2)
- net at M1.W4 (IGN8): now also J5.6 (Pin_6)
- net at M1.W5 (IGN7): now also J5.5 (Pin_5)
- net at M1.W6 (IGN6): now also J5.4 (Pin_4)
- net at M1.W7 (IGN5): now also J5.3 (Pin_3)
- net at J1.B21: now also R70.1
- net P1: now reaches J1.A31
- net P1: now also P1.1 (Pin_1)
- net +12V_PROT: now reaches M2.W5 (V12P)
- net +12V_PROT: now also RN3.5 (R4.2), RN3.6 (R3.2), RN3.7 (R2.2), RN3.8 (R1.2), RN4.5 (R4.2), RN4.6 (R3.2), RN4.7 (R2.2), RN4.8 (R1.2), RN5.5 (R4.2), RN5.6 (R3.2), RN5.7 (R2.2), RN5.8 (R1.2), RN6.5 (R4.2), RN6.6 (R3.2), RN6.7 (R2.2), RN7.5 (R4.2), RN7.6 (R3.2), RN7.7 (R2.2), RN7.8 (R1.2)
- net at M6.V2 (UART_RX): now also R6.2
- net LIN: now reaches M6.V4 (LIN)
- net LIN: now also R84.2
- net at M6.V5 (UART_TX): now also R7.2
- net P2: now reaches J1.B10
- net P2: now also P2.1 (Pin_1)
- net VTC_LS: now reaches M8.S1 (OUT_IGN8)
- net VTC_LS: now also Q6.1 (G), R29.1
- net LS_EVAP: now reaches M8.S2 (OUT_IGN7)
- net LS_EVAP: now also Q5.1 (G), R28.1
- net WBO_HEATER_LOW_SIDE: now reaches M8.S3 (OUT_IGN6)
- net WBO_HEATER_LOW_SIDE: now also Q3.1 (G), R26.1
- net AUX_LS1: now reaches M8.S4 (OUT_IGN5)
- net AUX_LS1: now also Q4.1 (G), R27.1
- net AUX_LS3: now reaches M8.S5 (OUT_IGN4)
- net AUX_LS3: now also Q1.1 (G), R24.1
- net AUX_LS2: now reaches M8.S6 (OUT_IGN3)
- net AUX_LS2: now also Q2.1 (G), R25.1
- net P16: now reaches M8.S7 (OUT_IGN2)
- net P16: now also P16.1 (Pin_1)
- net P15: now reaches M8.S8 (OUT_IGN1)
- net P15: now also P15.1 (Pin_1)
- net MCU_AUX_LS1: now reaches M8.V4 (IGN5)
- net MCU_AUX_LS1: now also RN2.5 (R4.2)
- net at M3.W5 (nReset): now also J4.5 (Pin_5)
- net at M3.W6 (SWDIO): now also J4.4 (Pin_4)
- net at M3.W7 (SWCLK): now also J4.2 (Pin_2)
- net at M3.W8 (V33_OUT): now also J4.1 (Pin_1)
- net at J1.B18: now also R69.1
- net P4: now reaches J1.B13
- net P4: now also P4.1 (Pin_1)
- net P13: now reaches J1.A22
- net P13: now also P13.1 (Pin_1)
- net at J1.A27: now also R59.1
- net at J1.B23: now also R72.1
- net at J1.B7: now also R65.1
- net at J1.B9: now also R67.1
- net at U2.8: now also R5.1
- net ALTERNATOR_CONTROL_LS: now reaches M2.S10 (OUT_LOW11)
- net ALTERNATOR_CONTROL_LS: now also D39.2 (A), D43.2 (K), R69.2
- net VTS_HS: now reaches M2.S12 (OUT_LOW8_PULLUP)
- net VTS_HS: now also U5.2 (IN), U6.2 (IN)
- net OUT_IDLE_AIR: now reaches M2.S15 (OUT_INJ6)
- net OUT_IDLE_AIR: now also D22.2 (A), D26.2 (K), D4.2 (A), R49.2
- net OUT_TACHOMETER: now reaches M2.S6 (OUT_PP2)
- net OUT_TACHOMETER: now also D38.2 (A), D42.2 (K), R85.2
- net P19: now reaches M2.S7 (OUT_LOW3_DUAL)
- net P19: now also P19.1 (Pin_1)
- net OUT_RADIATOR_RELAY: now reaches M2.S8 (OUT_LOW1)
- net OUT_RADIATOR_RELAY: now also D45.2 (A), D49.2 (K), R64.2
- net OUT_FUEL_RELAY: now reaches M2.W1 (OUT_LOW2)
- net OUT_FUEL_RELAY: now also D46.2 (A), D50.2 (K), R79.2
- net OUT_AC_LS: now reaches M2.W10 (OUT_INJ5)
- net OUT_AC_LS: now also D21.2 (A), D25.2 (K), D5.2 (A), R82.2
- net OUT_LOCKOUT_SOLENOID: now reaches M2.W11 (OUT_INJ8)
- net OUT_LOCKOUT_SOLENOID: now also D2.2 (A), D24.2 (A), D28.2 (K), R65.2
- net OUT_INTAKE_RUNNER: now reaches M2.W12 (OUT_INJ7)
- net OUT_INTAKE_RUNNER: now also D23.2 (A), D27.2 (K), D3.2 (A), R71.2
- net OUT_MAIN_RELAY_CONTROL: now reaches M2.W13 (OUT_LOW5_MAIN)
- net OUT_MAIN_RELAY_CONTROL: now also D48.2 (A), D52.2 (K), R80.2
- net WBO_RELAY_OUTPUT_LS: now reaches M2.W2 (OUT_LOW10)
- net WBO_RELAY_OUTPUT_LS: now also D47.2 (A), D51.2 (K), R81.2
- net P21: now reaches M2.W3 (OUT_LOW6_DIODE)
- net P21: now also P21.1 (Pin_1)
- net P20: now reaches M2.W4 (OUT_LOW4_DUAL)
- net P20: now also P20.1 (Pin_1)
- net P18: now reaches M2.W6 (OUT_PP1)
- net P18: now also P18.1 (Pin_1)
- net P23: now reaches M2.W8 (OUT_HIGH1)
- net P23: now also P23.1 (Pin_1)
- net P22: now reaches M2.W9 (OUT_LOW7_PULLUP)
- net P22: now also P22.1 (Pin_1)
- removed net 5V_SENSOR_1: J1.A20, J1.A21, J1.E5
- net IN_CAM1: no longer names the net of J1.A19
- net IN_CAM1: now also R52.1
- net IN_CAM_SYNC: no longer names the net of J1.A26
- net IN_CAM_SYNC: now also R58.1; no longer M1.S14 (IN_RES2)
- net IN_CRANK: no longer names the net of J1.A7
- net IN_CRANK: now also R47.1; no longer M1.S17 (IN_RES1)
- net IN_MRC: no longer names the net of J1.B22
- net IN_MRC: now also R71.1
- net IN_VTPSW renamed P3
- net P3: now also P3.1 (Pin_1)
- net IN_VVT_CAM: no longer names the net of J1.A25
- net IN_VVT_CAM: now also R57.1; no longer M1.S18 (IN_RES3)
- net OUT_ETB_RELAY: no longer names the net of J1.D15
- net OUT_FUEL_PUMP: no longer names the net of J1.E17
- net OUT_MAIN: no longer names the net of J1.E7
- net OUT_MAIN: now also R80.1
- net OUT_MCS renamed OUT_VTS_HS
- net OUT_VTS_HS: now also C12.1, D12.1 (K), D40.2 (A), D44.2 (K), R32.2, U5.1 (OUT), U5.5 (OUT), U6.3 (OUT)
- net OUT_VTC: no longer names the net of J1.B1
- net OUT_VTC: now also R63.1
- net OUT_VTS: no longer names the net of J1.B6
- net OUT_VTS: now also R64.1
- new net: J1.A6, R46.1
- new net: D21.1 (K), D25.1 (A), RN4.4 (R4.1)
- new net: D19.1 (K), D20.1 (A), RN3.1 (R1.1)
- new net: D48.1 (K), D52.1 (A), RN7.1 (R1.1)
- new net: D32.1 (K), D36.1 (A), RN5.1 (R1.1)
- new net: D37.1 (K), D41.1 (A), RN6.4 (R4.1)
- new net: R31.1, U6.4 (ST)
- new net: D40.1 (K), D44.1 (A), RN6.1 (R1.1)
- new net: J1.A8, R48.1
- new net: R30.2, U6.1 (GND)
- new net: J1.E22, R83.1
- new net: J1.E24, R84.1
- new net: J1.E31, R86.1
- new net: J1.E4, P6.1 (Pin_1)
- new net: D39.1 (K), D43.1 (A), RN6.2 (R2.1)
- new net: J1.A16, R50.1
- new net: D24.1 (K), D28.1 (A), RN4.1 (R1.1)
- new net: D23.1 (K), D27.1 (A), RN4.2 (R2.1)
- new net: R33.1, U5.4 (IS)
- new net: D17.1 (K), D18.1 (A), RN3.2 (R2.1)
- new net: D15.1 (K), D16.1 (A), RN3.3 (R3.1)
- new net: D13.1 (A), D14.1 (K), RN3.4 (R4.1)
- new net: D38.1 (K), D42.1 (A), RN6.3 (R3.1)
- new net: D47.1 (K), D51.1 (A), RN7.2 (R2.1)
- new net: D46.1 (K), D50.1 (A), RN7.3 (R3.1)
- new net: D45.1 (K), D49.1 (A), RN7.4 (R4.1)
- new net: J1.A18, R51.1
- new net: D29.1 (K), D33.1 (A), RN5.4 (R4.1)
- new net: J1.A9, R87.1
- new net: J1.A1, R45.1
- new net: D30.1 (K), D34.1 (A), RN5.3 (R3.1)
- new net: J1.A20, R53.1
- new net: J1.A21, R54.1
- new net: J1.A23, R55.1
- new net: J1.A24, R56.1
- new net: J1.A29, R61.1
- new net: J1.A30, R62.1
- new net: J1.B17, R68.1
- new net: J1.B8, R66.1
- new net: D22.1 (K), D26.1 (A), RN4.3 (R3.1)
- new net 4WIRE_DENSO_SIGNAL-: R50.2
- new net IN_CAM_SYNC_HALL: D30.2 (A), D34.2 (K), M1.S14 (IN_RES2), R58.2
- new net IN_CRANK_HALL: D29.2 (A), D33.2 (K), M1.S17 (IN_RES1), R47.2
- new net IN_VVT_CAM_HALL: D32.2 (A), D36.2 (K), M1.S18 (IN_RES3), R57.2
- new net OUT_LS_EVAP: D10.2 (A), Q5.2 (D), R70.2
- new net OUT_VTC_LS: D11.2 (A), Q6.2 (D), R72.2
- new net OUT_WBO_HEATER_LOW_SIDE: D8.2 (A), Q3.2 (D), R45.2
- no-connect marks 50 -> 76
Other:
- added sheet DENSO (denso.kicad_sch)
- note added: "EGR"
- note added: "NC"
- note added: "Secondary O2"
- moved on the sheet: M3, M6, M7, U1, U2
