File: khellen.kicad_pcb (KiCad board)
At the start: 4 copper layers, 149.8 x 159.2 mm, 182 parts, among them J1 1318612-1, J3 USB_B, J4 Conn_01x06, J5 Conn_01x06_Pin, J6 Conn_01x05_Pin, M1 Module-mega-mcu144-0.7, M2 Module-output-0.3, M3 Module-wbo-0.5, M4 Module-power_12and5V-0.3, M5 Module-knock-0.2, M6 Module-lin-0.1, M7 Module-stlink-0.1, M8 Module-ign8-0.2, Q1 VND14NV04TR-E, Q2 VND14NV04TR-E, Q3 VND14NV04TR-E, Q4 VND14NV04TR-E, Q5 VND14NV04TR-E, Q6 VND14NV04TR-E, U1 TLE9201SG, U2 DG470, U4 MCP6004, U5 BTS6143D

Commit message: Updated PCB
Parts:
- moved RN1 117.0 mm to (178.7, 116.5), turned to 180 degrees
- moved RN2 116.6 mm to (178.8, 125.0), turned to 90 degrees
- moved R5 78.6 mm to (251.8, 130.5), turned to 180 degrees
- moved R1 77.7 mm to (250.8, 128.0), turned to -90 degrees
- moved R34 17.3 mm to (204.2, 90.9), turned to -90 degrees
Routing:
- net /OUT_IDLE_AIR: track 1.71 -> 185.9 mm, vias 0 -> 10
- net /IN_VIGN: track 0.00 -> 164.5 mm, vias 0 -> 2
- net +12V: track 0.00 -> 155.5 mm, vias 0 -> 1
- net /ALTERNATOR_CONTROL_LS: track 1.71 -> 132.0 mm, vias 0 -> 2
- net +5VP: track 18.4 -> 146.6 mm, vias 0 -> 4
- net GNDA: track 0.00 -> 106.7 mm, vias 0 -> 4
- net Net-(D1-K): track 29.5 -> 123.8 mm, vias 0 -> 1
- net /IN_TPS: track 0.00 -> 92.2 mm, vias 0 -> 1
- net /OUT_RADIATOR_RELAY: track 1.71 -> 92.6 mm, vias 0 -> 1
- net /OUT_IGN3: track 0.00 -> 86.2 mm, vias 0 -> 2
- net /OUT_IGN1: track 0.00 -> 85.3 mm, vias 0 -> 1
- net +12V_RAW: track 245.9 -> 330.0 mm, vias 16 -> 18
- net /OUT_IGN2: track 0.00 -> 83.9 mm, vias 0 -> 2
- net +3V3: track 0.00 -> 82.4 mm, vias 0 -> 3
- net +5V: track 0.00 -> 79.9 mm, vias 0 -> 4
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